File: Hardware_Design/EmoeNAP/EmoeNAP.kicad_sch (KiCad schematic)
At the start: 126 parts, among them J1 Power, J2 10Hz to WIDEBAND, J3 10Hz to 1MHz, J4 Input, J5 10Hz to 100kHz, U1 OPA1612, U2 OPA1612, U3 OPA1612, U4 PS-12E05, U5 OPA1612, U6 OPA1679, U7 OPA1612, U8 OPA1612

Commit message: Update EmoeNAP design
Parts:
- removed J1: Power, Connector_JST:JST_XH_B3B-XH-A_1x03_P2.50mm_Vertical, symbol Connector_Generic:Conn_01x03
- added C65: 2.2uF, Capacitor_Tantalum_SMD:CP_EIA-3216-10_Kemet-I, symbol Device:CP_Small
- added C66, C67, C68, C69, C72, C73: 100pF, Capacitor_SMD:C_0402_1005Metric, symbol Device:C_Small
- added C70, C71: 0.1uF, Capacitor_SMD:C_0402_1005Metric, symbol Device:C_Small
- added J1: Battery, Connector_JST:JST_XA_B02B-XASK-1_1x02_P2.50mm_Vertical, symbol Connector_Generic:Conn_01x02
- added J6: GREEN, TestPoint:TestPoint_2Pads_Pitch2.54mm_Drill0.8mm, symbol Connector_Generic:Conn_01x02
- added J7: RED, TestPoint:TestPoint_2Pads_Pitch2.54mm_Drill0.8mm, symbol Connector_Generic:Conn_01x02
- added J8: USB_CHR, Connector_JST:JST_XA_B02B-XASK-1_1x02_P2.50mm_Vertical, symbol Connector_Generic:Conn_01x02
- added R12, R15, R18, R24, R3, R30, R34, R41: 1R, Resistor_SMD:R_0402_1005Metric, symbol Device:R_Small_US
- added R45, R46, R48, R49, R53, R54: 10k, Resistor_SMD:R_0402_1005Metric, symbol Device:R_Small_US
- added R47, R50, R52, R55: 1k, Resistor_SMD:R_0402_1005Metric, symbol Device:R_Small_US
- added R51: 2k, Resistor_SMD:R_0402_1005Metric, symbol Device:R_Small_US
- added RISO5, RISO6, RISO7: 100R, Resistor_SMD:R_0603_1608Metric, symbol Device:R_Small_US
- added U10: PS-12E05, EmoeNAP_FootPrint_Lib:PS-12E05, symbol NoiseAMP:PS-12E05
- added U11: TP4057, Package_TO_SOT_SMD:SOT-23-6, symbol Custom_Power:TP4057
- added U12: SGM321, Package_TO_SOT_SMD:SOT-23-5, symbol Amplifier_Operational:LM321
- added U9: LT1364, Package_SO:SOIC-8_3.9x4.9mm_P1.27mm, symbol Amplifier_Operational:LM358
- renumbered C51 to C50, C52 to C51, C53 to C52, C54 to C53, C56 to C54, C57 to C55, C58 to C56, C59 to C57, C60 to C58, C61 to C59, C62 to C60, C64 to C61, C65 to C62, C66 to C63, C67 to C64, R9 to R10, R10 to R11, R11 to R13, R12 to R14, R13 to R16, R14 to R17, R15 to R19, R16 to R20, R17 to R21, R18 to R22, R19 to R23, R20 to R25, R21 to R26, R22 to R27, R23 to R28, R24 to R29, R25 to R31, R26 to R32, R27 to R33, R28 to R35, R29 to R36, R30 to R37, R31 to R38, R32 to R39, R3 to R4, R33 to R40, R34 to R42, R35 to R43, R36 to R44, R4 to R5, R5 to R6, R6 to R7, R7 to R8, R8 to R9, TP4 to TP3, TP3 to TP4
Connections:
- net GND: now also C70.2, R47.1, R50.1, R55.1, RISO5.2, RISO6.2, RISO7.2
- net VDD: now also C65.1, C70.1, R45.2, R48.2, R53.2, U10.1, U12.5 (V+), U9.8 (V+)
- net VSS: now also C65.2, C66.2, C68.2, C71.1, C72.2, J1.2 (Pin_2), J8.2 (Pin_2), R46.1, R49.1, R51.2, R54.1, U10.4, U11.2 (GND), U12.2 (V-), U9.4 (V-)
- new net: R41.1, R44.1, U8.7
- new net: C1.1, R12.2, R15.2, R18.2, R24.2, R3.2, R30.2, R34.2, R41.2
- new net: R3.1, R9.1, U1.1
- new net: C68.1, R48.1, R49.2, U9.5 (+)
- new net: C73.2, RISO7.1, U12.4
- new net: C72.1, R53.1, R54.2, U12.1 (+)
- new net: C66.1, R45.1, R46.2, U9.3 (+)
- new net: J6.1 (Pin_1), J7.1 (Pin_1), R52.2
- new net: J7.2 (Pin_2), U11.1 (~{CHRG})
- new net: J6.2 (Pin_2), U11.5 (~{STDBY})
- new net: R51.1, U11.6 (PROG)
- new net: R24.1, R28.1, U7.1
- new net: C69.1, R50.2, U9.6 (-)
- new net: C69.2, RISO6.1, U9.7
- new net: C67.1, R47.2, U9.2 (-)
- new net: R30.1, R33.1, U7.7
- new net: C73.1, R55.2, U12.3 (-)
- new net: R18.1, R21.1, U5.7
- new net: C67.2, RISO5.1, U9.1
- new net: R15.1, R17.1, U5.1
- new net: R34.1, R40.1, U8.1
- new net: R12.1, R14.1, U1.7
- new net VBAT: J1.1 (Pin_1), U10.2
- new net VBAT_CHRG: U10.3, U11.3 (BAT)
- new net VBUS_+5V: C71.2, J8.1 (Pin_1), R52.1, U11.4 (Vcc)
Other:
- note added: "Assembly 1"
- note added: "Assembly 1 and 2 are two redundant backup."
- note added: "Assembly 2(Backup)"
- note added: "IMPORTANT:"
- note added: "Single Cell Li-ion Battery (+4.2V MAX)"
- note added: "Virtual Ground Generator from @CNPP"
- note added: "Virtual Ground circuit is more convenient to operate on single cell battery.But it intro- duces a lot of noise to system noise floor. For best noise floor performance, please use 2-cell battery to provide true bipolar power supply."
- note removed: "±5V Power Supply Maximum I = ±100mA"
- moved on the sheet: H1, H2, H3, H4, R19

Commit message: Update progress and notes
Parts:
- RISO3: value 10R -> 0R
Other:
- note added: "Virtual Ground circuit is more convenient to operate on single cell battery.But it intro- duces a little noise to system noise floor. For best noise floor performance, please use 2-cell battery to provide true bipolar power supply."
- note removed: "Virtual Ground circuit is more convenient to operate on single cell battery.But it intro- duces a lot of noise to system noise floor. For best noise floor performance, please use 2-cell battery to provide true bipolar power supply."
Changed lines of the file:
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@@
     (effects (font (size 2.0066 2.0066)) (justify left bottom))
   )
-  (text "	Virtual Ground circuit is more convenient\nto operate on single cell battery.But it intro-\nduces a lot of noise to system noise floor.\n	For best noise floor performance, please \nuse 2-cell battery to provide true bipolar \npower supply."
+  (text "	Virtual Ground circuit is more convenient\nto operate on single cell battery.But it intro-\nduces a little noise to system noise floor.\n	For best noise floor performance, please \nuse 2-cell battery to provide true bipolar \npower supply."
     (at 107.95 270.51 0)
     (effects (font (size 2 2) (thickness 0.4) bold italic) (justify left bottom))
@@
       (effects (font (size 1.27 1.27)) (justify left))
     )
-    (property "Value" "10R" (at 71.12 160.02 0)
+    (property "Value" "0R" (at 71.12 160.02 0)
       (effects (font (size 1.27 1.27)) (justify left))
     )
