File: Hardware_Design/NoiseAMP_BAT/NoiseAMP_BAT.kicad_sch (KiCad schematic)
At the start: 23 parts, among them J1 VIN, J2 SW, J3 PWR, J4 LED, J5 SW, U1 IP2325, U2 Bat_Pack

Commit message: Update EmoeNAP design
Connections:
- net Common: now reaches J3.2 (Pin_2), U2.2 (-), U2.3 (+)
Changed lines of the file:
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@@
   (junction (at 189.23 85.09) (diameter 0) (color 0 0 0 0)
   )
+  (junction (at 106.68 92.71) (diameter 0) (color 0 0 0 0)
+  )
   (junction (at 213.36 95.25) (diameter 0) (color 0 0 0 0)
   )
@@
     (stroke (width 0) (type default) (color 0 0 0 0))
   )
+  (wire (pts (xy 106.68 92.71) (xy 113.03 92.71))
+    (stroke (width 0) (type default) (color 0 0 0 0))
+  )
   (wire (pts (xy 165.1 85.09) (xy 154.94 85.09))
     (stroke (width 0) (type default) (color 0 0 0 0))
@@
     (stroke (width 0) (type default) (color 0 0 0 0))
   )
+  (label "Common" (at 113.03 92.71 0)
+    (effects (font (size 1.27 1.27)) (justify left bottom))
+  )
   (symbol (lib_id "Device:C_Small") (at 140.97 93.98 0) (unit 1)
